Commit message: fix: PointCloud direction and Lidar coordinate.

File: src/autoracer_robot_urdf/urdf/autoracer.urdf.xacro (robot description, xacro)
@@ -42,5 +42,5 @@
   <xacro:property name="lidar_x" value="0.24"/>
   <xacro:property name="lidar_z" value="0.39"/>
-  <xacro:property name="lidar_yaw" value="1.5708"/>
+  <xacro:property name="lidar_yaw" value="-1.5708"/>
   <xacro:property name="zed_x" value="0.34"/>
   <xacro:property name="zed_z" value="0.29"/>

Commit message: chore: save current integration state, mapping pending test

File: src/autoracer_robot_urdf/urdf/autoracer.urdf.xacro (robot description, xacro)
@@ -14,4 +14,6 @@
 -->
 <robot xmlns:xacro="http://www.ros.org/wiki/xacro" name="autoracer">
+  <xacro:arg name="prefix" default=""/>
+  <xacro:property name="prefix" value="$(arg prefix)"/>
   <!-- ==================== 参数定义 ==================== -->
   <!-- 底盘尺寸 -->
@@ -95,5 +97,5 @@
   </xacro:macro>
   <!-- ==================== base_link (后轴中心，轴高度) ==================== -->
-  <link name="base_link">
+  <link name="${prefix}base_link">
     <inertial>
       <origin xyz="${chassis_x_offset} 0 ${chassis_z_offset + chassis_height/2.0}" rpy="0 0 0"/>
@@ -117,22 +119,22 @@
   <!-- ==================== 后轮 (continuous joints) ==================== -->
   <!-- 左后轮 -->
-  <xacro:wheel_link name="rear_left_wheel_link"/>
-  <joint name="rear_left_wheel_joint" type="continuous">
+  <xacro:wheel_link name="${prefix}rear_left_wheel_link"/>
+  <joint name="${prefix}rear_left_wheel_joint" type="continuous">
     <origin xyz="0 ${track_width/2.0} 0" rpy="0 0 0"/>
-    <parent link="base_link"/>
-    <child link="rear_left_wheel_link"/>
+    <parent link="${prefix}base_link"/>
+    <child link="${prefix}rear_left_wheel_link"/>
     <axis xyz="0 1 0"/>
   </joint>
   <!-- 右后轮 -->
-  <xacro:wheel_link name="rear_right_wheel_link"/>
-  <joint name="rear_right_wheel_joint" type="continuous">
+  <xacro:wheel_link name="${prefix}rear_right_wheel_link"/>
+  <joint name="${prefix}rear_right_wheel_joint" type="continuous">
     <origin xyz="0 ${-track_width/2.0} 0" rpy="0 0 0"/>
-    <parent link="base_link"/>
-    <child link="rear_right_wheel_link"/>
+    <parent link="${prefix}base_link"/>
+    <child link="${prefix}rear_right_wheel_link"/>
     <axis xyz="0 1 0"/>
   </joint>
   <!-- ==================== 前轮转向 (revolute + continuous) ==================== -->
   <!-- 左前转向节 -->
-  <link name="front_left_steering_link">
+  <link name="${prefix}front_left_steering_link">
     <inertial>
       <origin xyz="0 0 0" rpy="0 0 0"/>
@@ -148,21 +150,21 @@
     </visual>
   </link>
-  <joint name="front_left_steering_joint" type="revolute">
+  <joint name="${prefix}front_left_steering_joint" type="revolute">
     <origin xyz="${wheelbase} ${track_width/2.0} 0" rpy="0 0 0"/>
-    <parent link="base_link"/>
-    <child link="front_left_steering_link"/>
+    <parent link="${prefix}base_link"/>
+    <child link="${prefix}front_left_steering_link"/>
     <axis xyz="0 0 1"/>
     <limit lower="${-max_steering_angle}" upper="${max_steering_angle}" effort="10" velocity="1.0"/>
   </joint>
   <!-- 左前轮 -->
-  <xacro:wheel_link name="front_left_wheel_link"/>
-  <joint name="front_left_wheel_joint" type="continuous">
+  <xacro:wheel_link name="${prefix}front_left_wheel_link"/>
+  <joint name="${prefix}front_left_wheel_joint" type="continuous">
     <origin xyz="0 0 0" rpy="0 0 0"/>
-    <parent link="front_left_steering_link"/>
-    <child link="front_left_wheel_link"/>
+    <parent link="${prefix}front_left_steering_link"/>
+    <child link="${prefix}front_left_wheel_link"/>
     <axis xyz="0 1 0"/>
   </joint>
   <!-- 右前转向节 -->
-  <link name="front_right_steering_link">
+  <link name="${prefix}front_right_steering_link">
     <inertial>
       <origin xyz="0 0 0" rpy="0 0 0"/>
@@ -178,22 +180,22 @@
     </visual>
   </link>
-  <joint name="front_right_steering_joint" type="revolute">
+  <joint name="${prefix}front_right_steering_joint" type="revolute">
     <origin xyz="${wheelbase} ${-track_width/2.0} 0" rpy="0 0 0"/>
-    <parent link="base_link"/>
-    <child link="front_right_steering_link"/>
+    <parent link="${prefix}base_link"/>
+    <child link="${prefix}front_right_steering_link"/>
     <axis xyz="0 0 1"/>
     <limit lower="${-max_steering_angle}" upper="${max_steering_angle}" effort="10" velocity="1.0"/>
   </joint>
   <!-- 右前轮 -->
-  <xacro:wheel_link name="front_right_wheel_link"/>
-  <joint name="front_right_wheel_joint" type="continuous">
+  <xacro:wheel_link name="${prefix}front_right_wheel_link"/>
+  <joint name="${prefix}front_right_wheel_joint" type="continuous">
     <origin xyz="0 0 0" rpy="0 0 0"/>
-    <parent link="front_right_steering_link"/>
-    <child link="front_right_wheel_link"/>
+    <parent link="${prefix}front_right_steering_link"/>
+    <child link="${prefix}front_right_wheel_link"/>
     <axis xyz="0 1 0"/>
   </joint>
   <!-- ==================== 传感器 link ==================== -->
   <!-- LiDAR C32 (固定在 base_link 上) -->
-  <link name="laser">
+  <link name="${prefix}laser">
     <inertial>
       <origin xyz="0 0 0" rpy="0 0 0"/>
@@ -215,11 +217,11 @@
     </collision>
   </link>
-  <joint name="laser_joint" type="fixed">
+  <joint name="${prefix}laser_joint" type="fixed">
     <origin xyz="${lidar_x} 0 ${lidar_z}" rpy="0 0 ${lidar_yaw}"/>
-    <parent link="base_link"/>
-    <child link="laser"/>
+    <parent link="${prefix}base_link"/>
+    <child link="${prefix}laser"/>
   </joint>
   <!-- ZED X 深度相机 (固定在 base_link 上) -->
-  <link name="zed_camera_link">
+  <link name="${prefix}zed_camera_link">
     <inertial>
       <origin xyz="0 0 0" rpy="0 0 0"/>
@@ -241,8 +243,8 @@
     </collision>
   </link>
-  <joint name="zed_camera_joint" type="fixed">
+  <joint name="${prefix}zed_camera_joint" type="fixed">
     <origin xyz="${zed_x} 0 ${zed_z}" rpy="0 0 0"/>
-    <parent link="base_link"/>
-    <child link="zed_camera_link"/>
+    <parent link="${prefix}base_link"/>
+    <child link="${prefix}zed_camera_link"/>
   </joint>
 </robot>

Commit message: Make stage one handoff verifiable before path tracking
Stage one now has calibrated Hall odometry, wheel/IMU EKF wiring, static IMU TF, bringup launch entry points, acceptance checks, and the live low-speed rosbag evidence used for independent verification. The path tracking fixtures are kept in the same handoff so phase two starts from a reproducible baseline rather than an untracked workspace.

Constraint: Stage one PASS requires decoded telemetry, fused odom, motion proof, and independent verifier evidence

Rejected: Commit only source code without rosbag evidence | would leave the live hard-pass run unverifiable after push

Confidence: high

Scope-risk: moderate

Directive: Do not claim stage two live PASS from this commit; only offline fixtures are covered

Tested: colcon build --symlink-install --packages-up-to autoracer_bringup turn_on_autoracer_robot hipnuc_imu

Tested: python3 tools/acceptance/stage1_acceptance_check.py --mode offline

Tested: ros2 bag info docs/test-records/rosbags/stage1-hardpass-2026-05-15-0p5mps

Not-tested: Stage two live path tracking on the vehicle

File: src/autoracer_robot_urdf/urdf/autoracer.urdf.xacro (robot description, xacro)
@@ -8,5 +8,5 @@
   实测参数 (2026-01-29):
     车辆: 长0.85m, 宽0.50m, 高0.40m
-    轴距: 0.54m (前轴距车头0.15m, 后轴距车尾0.16m)
+    轴距: 0.60m (前轴距车头0.15m, 后轴距车尾0.16m)
     轮距: 0.48m
     轮径: 0.11m (半径)
@@ -22,5 +22,5 @@
   <xacro:property name="chassis_height" value="0.20"/>
   <!-- Ackermann 运动学参数 -->
-  <xacro:property name="wheelbase" value="0.54"/>
+  <xacro:property name="wheelbase" value="0.60"/>
   <xacro:property name="track_width" value="0.48"/>
   <xacro:property name="wheel_radius" value="0.11"/>

Commit message: Calibrate steering limits against measured vehicle geometry
The front-to-rear wheelbase is confirmed at 0.60 m and the Hall wheel diameter remains 0.235 m, so the ROS geometry, URDF axle height, planner constraints, and tracker clamps now use a 0.262 rad steering limit and a 2.24 m minimum turning radius. The left/right stage-2 arc fixtures move to 2.5 m so the acceptance path stays feasible under the measured 15 degree steering limit.

Constraint: Positive steering remains left turn per the existing Ackermann protocol
Constraint: Servo endpoints are measured as 1105 us and 1895 us around a provisional 1500 us center
Rejected: Keep the old 0.393 rad steering limit | it implied a 1.45 m turning radius the measured steering cannot support
Confidence: high
Scope-risk: moderate
Directive: Do not change wheel radius independently of the confirmed 0.235 m wheel diameter
Tested: python3 tools/acceptance/stage1_acceptance_check.py --mode offline; python3 tools/acceptance/stage2_path_fixture_check.py; python3 tools/acceptance/stage2_tracker_fake_odom_check.py; colcon build --symlink-install --packages-select turn_on_autoracer_robot autoracer_path_tracking autoracer_bringup autoracer_robot_urdf autoracer_robot_nav2
Not-tested: Windows/Keil firmware build or real-car steering sweep after flashing
Co-authored-by: OmX <omx@oh-my-codex.dev>

File: src/autoracer_robot_urdf/urdf/autoracer.urdf.xacro (robot description, xacro)
@@ -5,11 +5,11 @@
   坐标系约定 (ROS REP-103):
     X = 前, Y = 左, Z = 上
-    base_link = 后轴中心，轴高度 (Z=0.11m above ground)
-  实测参数 (2026-01-29):
-    车辆: 长0.85m, 宽0.50m, 高0.40m
+    base_link = 后轴中心，轴高度 (Z=0.1175m above ground)
+  当前参数 (2026-05-15 calibration update):
+    车辆外廓: 长0.85m, 宽0.50m, 总高0.40m；URDF 底盘盒高0.20m
     轴距: 0.60m (前轴距车头0.15m, 后轴距车尾0.16m)
-    轮距: 0.48m
-    轮径: 0.11m (半径)
-    最大转向角: 0.393 rad (≈22.5°)
+    轮距: 0.48m (待复核)
+    轮径: 0.235m (半径0.1175m)
+    最大转向角: 0.262 rad (≈15°)
 -->
 <robot xmlns:xacro="http://www.ros.org/wiki/xacro" name="autoracer">
@@ -24,7 +24,7 @@
   <xacro:property name="wheelbase" value="0.60"/>
   <xacro:property name="track_width" value="0.48"/>
-  <xacro:property name="wheel_radius" value="0.11"/>
+  <xacro:property name="wheel_radius" value="0.1175"/>
   <xacro:property name="wheel_width" value="0.08"/>
-  <xacro:property name="max_steering_angle" value="0.393"/>
+  <xacro:property name="max_steering_angle" value="0.262"/>
   <!-- 底盘布局 (base_link 在后轴中心) -->
   <xacro:property name="front_axle_to_front" value="0.15"/>

Commit message: Reconcile vehicle envelope with measured track and overhangs
The latest chassis measurements confirm a 0.47 m track width, a 0.57 m collision width, a 0.16 m rear overhang, and a front collision edge defined by the front wheel radius rather than the bumper. The URDF geometry, Nav2 costmap footprint, package docs, and LIO-SAM reference translation now use a 0.8775 m by 0.57 m vehicle envelope while keeping total height and sensor extrinsics marked for final installation recheck.

Constraint: Front wheels extend beyond the front bumper, so the navigation footprint front edge is wheelbase plus wheel radius
Rejected: Keep the old 0.85 m by 0.50 m footprint | it no longer bounds the measured vehicle width or front wheel protrusion
Confidence: high
Scope-risk: moderate
Directive: Do not shrink the Nav2 footprint unless a new physical collision-envelope measurement replaces the 2026-05-15 values
Tested: python3 tools/acceptance/stage2_path_fixture_check.py; python3 tools/acceptance/stage2_tracker_fake_odom_check.py; colcon build --symlink-install --packages-select autoracer_robot_urdf autoracer_robot_nav2; git diff --cached --check
Not-tested: lio_sam package build because GTSAM is not installed on this machine; real Nav2 obstacle clearance with the updated footprint
Co-authored-by: OmX <omx@oh-my-codex.dev>

File: src/autoracer_robot_urdf/urdf/autoracer.urdf.xacro (robot description, xacro)
@@ -7,7 +7,7 @@
     base_link = 后轴中心，轴高度 (Z=0.1175m above ground)
   当前参数 (2026-05-15 calibration update):
-    车辆外廓: 长0.85m, 宽0.50m, 总高0.40m；URDF 底盘盒高0.20m
-    轴距: 0.60m (前轴距车头0.15m, 后轴距车尾0.16m)
-    轮距: 0.48m (待复核)
+    车辆碰撞外廓: 长0.8775m, 宽0.57m；总高待复核；URDF 底盘盒高0.20m
+    轴距: 0.60m (前轮最前点距前轴0.1175m, 后轴距车尾0.16m)
+    轮距: 0.47m
     轮径: 0.235m (半径0.1175m)
     最大转向角: 0.262 rad (≈15°)
@@ -18,15 +18,15 @@
   <!-- ==================== 参数定义 ==================== -->
   <!-- 底盘尺寸 -->
-  <xacro:property name="chassis_length" value="0.85"/>
-  <xacro:property name="chassis_width" value="0.50"/>
+  <xacro:property name="chassis_length" value="0.8775"/>
+  <xacro:property name="chassis_width" value="0.57"/>
   <xacro:property name="chassis_height" value="0.20"/>
   <!-- Ackermann 运动学参数 -->
   <xacro:property name="wheelbase" value="0.60"/>
-  <xacro:property name="track_width" value="0.48"/>
+  <xacro:property name="track_width" value="0.47"/>
   <xacro:property name="wheel_radius" value="0.1175"/>
   <xacro:property name="wheel_width" value="0.08"/>
   <xacro:property name="max_steering_angle" value="0.262"/>
   <!-- 底盘布局 (base_link 在后轴中心) -->
-  <xacro:property name="front_axle_to_front" value="0.15"/>
+  <xacro:property name="front_axle_to_front" value="0.1175"/>
   <xacro:property name="rear_axle_to_rear" value="0.16"/>
   <!-- base_link 高度 (轴心离地高度) -->
